Commit message: Vertical movement done

File: dronefiles/src/tello_ros/tello_description/urdf/tello.xacro (robot description, xacro)
@@ -2,5 +2,7 @@
 <!-- Body coordinates are: x forward, y left, z up; rotation is: roll right, pitch forward, yaw left -->
 <!-- See http://www.ros.org/reps/rep-0103.html -->
-<robot name="tello${suffix}">
+<robot xmlns:xacro="http://ros.org/wiki/xacro" name="tello">
+    <xacro:arg name="suffix" default=""/>
+    <xacro:arg name="topic_ns" default="tello"/>
     <!-- Materials -->
     <material name="gray">
@@ -15,5 +17,5 @@
     <!-- TODO add Gazebo color information -->
     <!-- Base link -->
-    <link name="base_link${suffix}">
+    <link name="base_link">
         <visual>
             <origin xyz="0 0 0.01"/>
@@ -70,5 +72,5 @@
     </link>
     <!-- Camera link -->
-    <link name="camera_link${suffix}">
+    <link name="camera_link">
         <visual>
             <origin xyz="0 0 0"/>
@@ -89,15 +91,15 @@
     </link>
     <!-- Fixed joint -->
-    <joint name="camera_joint${suffix}" type="fixed">
+    <joint name="camera_joint" type="fixed">
         <origin xyz="0.035 0 0" rpy="0 0 0"/>  <!-- TODO fix origin -->
-        <parent link="base_link${suffix}"/>
-        <child link="camera_link${suffix}"/>
+        <parent link="base_link"/>
+        <child link="camera_link"/>
     </joint>
     <!-- Tello plugin for Gazebo -->
     <gazebo>
         <plugin name="TelloPlugin" filename="libTelloPlugin.so">
-            <namespace>${topic_ns}</namespace>
+            <namespace>"topic_ns"</namespace>
             <parameter name="use_sim_time" type="bool">1</parameter>
-            <link_name>base_link${suffix}</link_name>
+            <link_name>base_link</link_name>
             <center_of_mass>0 0 0</center_of_mass>
         </plugin>
@@ -106,6 +108,6 @@
     <!-- TODO use Tello camera specs -->
     <!-- TODO add another joint and rotate the camera into place -->
-    <gazebo reference="camera_link${suffix}">
-        <sensor type="camera" name="${topic_ns}">
+    <gazebo reference="camera_link">
+        <sensor type="camera" name="topic_ns">
             <update_rate>30.0</update_rate>
             <camera name="head">  <!-- TODO does this name do anything? -->
@@ -129,5 +131,5 @@
                 </noise>
             </camera>
-            <plugin name="camera_controller${suffix}" filename="libgazebo_ros_camera.so">
+            <plugin name="camera_controller" filename="libgazebo_ros_camera.so">
                 <alwaysOn>true</alwaysOn>
                 <updateRate>0.0</updateRate>
@@ -135,5 +137,5 @@
                 <imageTopicName>image_raw</imageTopicName>
                 <cameraInfoTopicName>camera_info</cameraInfoTopicName>
-                <frameName>camera_link${suffix}</frameName>
+                <frameName>camera_link</frameName>
                 <hackBaseline>0.07</hackBaseline>
                 <distortionK1>0.0</distortionK1>
